File: PicoLink.kicad_pcb (KiCad board)
At the start: 2 copper layers, 34 x 60.1 mm, 51 parts, among them J1 USB_C_Receptacle_USB2.0_16P, J3 DE15_Pins_HighDensity_Mountin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, J4 RAHPCUA20, J6 Conn_01x14_Pin, J7 Conn_01x14_Pin, J8 Conn_01x14_Pin, J9 Conn_01x14_Pin, SW2 SW_Push, SW3 SW_Push, SW4 SW_Push, SW5 SW_Push, U1 RP2040, U2 AMS1117-3.3, U5 W25Q32JVSS, Y2 Crystal

Commit message: Fixed traces and added logo
Parts:
- removed Y2: Crystal, Crystal:Crystal_SMD_5032-2Pin_5.0x3.2mm
- removed kibuzzard-6A7FFE0F: G***, kibuzzard-6A7FFE0F
- removed kibuzzard-6A7FFE19: G***, kibuzzard-6A7FFE19
- added G***: LOGO, LOGO, B.Cu at (193.2, 123.3)
- added R12: 27.4, Resistor_SMD:R_0805_2012Metric, F.Cu at (196.6, 100.8)
- added R13: 27.4, Resistor_SMD:R_0805_2012Metric, F.Cu at (198.5, 100.8)
- added Y1: Crystal_GND24, Crystal:Crystal_SMD_Abracon_ABM8AIG-4Pin_3.2x2.5mm, F.Cu at (197.0, 123.5)
- added kibuzzard-6A81CC73: G***, kibuzzard-6A81CC73, B.Cu at (198.0, 91.0)
- added kibuzzard-6A81CC8C: G***, kibuzzard-6A81CC8C, B.Cu at (197.8, 96.5)
- added kibuzzard-6A81CC96: G***, kibuzzard-6A81CC96, B.Cu at (197.5, 100.7)
- R17, R6: value 330 -> 330R
Connections:
- U1 pad 46: /USB_D- -> Net-(U1-USB_DM)
- U1 pad 47: /USB_D+ -> Net-(U1-USB_DP)
Routing:
- net /USB_D+: track 47.9 -> 36.1 mm, vias 2 -> 0
- net /USB_D-: track 46.5 -> 35.4 mm, vias 4 -> 2
- net GND: track 78.0 -> 87.1 mm, vias 37 -> 39
- net Net-(U1-USB_DM): track 0.00 -> 9.11 mm, vias 0 -> 2
- net Net-(U1-USB_DP): track 0.00 -> 8.35 mm, vias 0 -> 2
- net +3V3: track 114.4 -> 111.6 mm, vias 15 -> 13
- net /IOVDD: track 133.1 -> 135.2 mm, vias 6 -> 5
- net /XIN: track 28.8 -> 30.6 mm
- net /+5V: track 55.9 -> 57.6 mm
- net /QSPI_SD2: track 105.1 -> 106.5 mm
- net /QSPI_SCLK: track 98.7 -> 97.6 mm
- net Net-(C13-Pad2): track 7.75 -> 8.85 mm
- net /IO5: track 22.9 -> 23.8 mm
- net /QSPI_SD0: track 38.1 -> 37.2 mm
- net /IO0: track 24.0 -> 23.3 mm
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