File: PicoLink.kicad_sch (KiCad schematic)
At the start: 42 parts, among them J1 USB_C_Receptacle_USB2.0_16P, J3 DE15_Pins_HighDensity_Mountin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, J4 RAHPCUA20, J6 Conn_01x14_Pin, J7 Conn_01x14_Pin, J8 Conn_01x14_Pin, J9 Conn_01x14_Pin, SW2 SW_Push, SW3 SW_Push, SW4 SW_Push, SW5 SW_Push, U1 RP2040, U2 AMS1117-3.3, U5 W25Q32JVSS, Y2 Crystal

Commit message: Fixed traces and added logo
Parts:
- removed Y2: Crystal, Crystal:Crystal_SMD_5032-2Pin_5.0x3.2mm, symbol Device:Crystal
- added R12, R13: 27.4, Resistor_SMD:R_0805_2012Metric, symbol Device:R
- added Y1: Crystal_GND24, Crystal:Crystal_SMD_Abracon_ABM8AIG-4Pin_3.2x2.5mm, symbol Device:Crystal_GND24
Connections:
- net GND: now also Y1.2 (G), Y1.4 (G)
- net USB_D+: now also R12.1; no longer U1.47 (USB_DP)
- net USB_D-: now also R13.1; no longer U1.46 (USB_DM)
- net XIN: now also Y1.1
- net at C13.2, R5.1: now also Y1.3
- new net: R12.2, U1.47 (USB_DP)
- new net: R13.2, U1.46 (USB_DM)
