File: PCB Files/PicoLink.kicad_pcb (KiCad board)
At the start: 2 copper layers, 34 x 60.1 mm, 55 parts, among them J1 USB_C_Receptacle_USB2.0_16P, J3 DE15_Pins_HighDensity_Mountin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, J4 RAHPCUA20, J6 Conn_01x14_Pin, J7 Conn_01x14_Pin, J8 Conn_01x14_Pin, J9 Conn_01x14_Pin, SW2 SW_Push, SW3 SW_Push, SW4 SW_Push, SW5 SW_Push, U1 RP2040, U2 AMS1117-3.3, U5 W25Q32JVSS, Y1 Crystal_GND24

Commit message: Changed some constraints
Parts:
- moved D1 1.65 mm to (208.5, 92.9)
Routing:
- net GND: track 87.1 -> 63.2 mm, vias 39 -> 31
- net /QSPI_SCLK: track 97.6 -> 88.5 mm
- net /IOVDD: track 135.2 -> 140.8 mm
- net +3V3: track 111.6 -> 106.3 mm, vias 13 -> 11
- net /SWDIO: track 23.7 -> 28.3 mm
- net Net-(U1-USB_DP): track 8.35 -> 12.5 mm
- net /IO5: track 23.8 -> 19.7 mm
- net /QSPI_SD3: track 97.8 -> 93.8 mm
- net /+5V: track 57.6 -> 54.1 mm
- net /QSPI_SD1: track 91.9 -> 94.3 mm
- net /ADC0: track 20.9 -> 23.3 mm
- net /HSYNC: track 26.1 -> 28.4 mm
- net /QSPI_SD2: track 106.5 -> 104.5 mm, vias 10 -> 8
- net Net-(U1-USB_DM): track 9.11 -> 10.9 mm
- net /VSYNC: track 24.6 -> 26.4 mm
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Other:
- board text removed: "IO5"
